File: LSM6DSL.kicad_pcb (KiCad board)
At the start: 2 copper layers, 25.4 x 14 mm, 6 parts, among them J1 Conn_01x10, U1 LSM6DSL

Commit message: Increased size
Other:
- board size 25.4 x 14 mm -> 26.4 x 14.5 mm
Changed lines of the file:
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@@
     (links 20)
     (no_connects 0)
-    (area 126.924999 112.954999 152.475001 127.075001)
+    (area 126.416999 112.954999 152.983001 127.583001)
     (thickness 1.6)
     (drawings 46)
@@
   (page A4)
   (layers
-    (0 F.Cu signal)
+    (0 F.Cu signal hide)
     (31 B.Cu signal)
     (32 B.Adhes user)
@@
     (34 B.Paste user)
     (35 F.Paste user)
-    (36 B.SilkS user)
-    (37 F.SilkS user)
+    (36 B.SilkS user hide)
+    (37 F.SilkS user hide)
     (38 B.Mask user)
     (39 F.Mask user)
@@
     (47 F.CrtYd user)
     (48 B.Fab user)
-    (49 F.Fab user)
+    (49 F.Fab user hide)
   )
   (setup
@@
     (pad_to_mask_clearance 0.0508)
     (aux_axis_origin 0 0)
-    (visible_elements FFFFFF7F)
+    (visible_elements 7FFFFDFF)
     (pcbplotparams
       (layerselection 0x00030_80000001)
@@
       (net 9 SDO-SA0))
   )
-  (gr_arc (start 128.27 114.3) (end 127 114.3) (angle 90) (layer Edge.Cuts) (width 0.15))
-  (gr_arc (start 151.13 114.3) (end 151.13 113.03) (angle 90) (layer Edge.Cuts) (width 0.15))
-  (gr_arc (start 151.13 125.73) (end 152.4 125.73) (angle 90) (layer Edge.Cuts) (width 0.15))
-  (gr_arc (start 128.27 125.73) (end 128.27 127) (angle 90) (layer Edge.Cuts) (width 0.15))
-  (dimension 25.4 (width 0.3) (layer Eco1.User)
-    (gr_text "25,400 mm" (at 139.7 131.75) (layer Eco1.User)
+  (dimension 26.416 (width 0.3) (layer Eco1.User)
+    (gr_text "26,416 mm" (at 139.7 132.668) (layer Eco1.User)
       (effects (font (size 1.5 1.5) (thickness 0.3)))
     )
-    (feature1 (pts (xy 152.4 128.4) (xy 152.4 133.1)))
-    (feature2 (pts (xy 127 128.4) (xy 127 133.1)))
-    (crossbar (pts (xy 127 130.4) (xy 152.4 130.4)))
-    (arrow1a (pts (xy 152.4 130.4) (xy 151.273496 130.986421)))
-    (arrow1b (pts (xy 152.4 130.4) (xy 151.273496 129.813579)))
-    (arrow2a (pts (xy 127 130.4) (xy 128.126504 130.986421)))
-    (arrow2b (pts (xy 127 130.4) (xy 128.126504 129.813579)))
-  )
-  (dimension 14 (width 0.3) (layer Eco1.User)
-    (gr_text "14,000 mm" (at 157.95 120 90) (layer Eco1.User)
+    (feature1 (pts (xy 126.492 128.778) (xy 126.492 134.018)))
+    (feature2 (pts (xy 152.908 128.778) (xy 152.908 134.018)))
+    (crossbar (pts (xy 152.908 131.318) (xy 126.492 131.318)))
+    (arrow1a (pts (xy 126.492 131.318) (xy 127.618504 130.731579)))
+    (arrow1b (pts (xy 126.492 131.318) (xy 127.618504 131.904421)))
+    (arrow2a (pts (xy 152.908 131.318) (xy 151.781496 130.731579)))
+    (arrow2b (pts (xy 152.908 131.318) (xy 151.781496 131.904421)))
+  )
+  (dimension 14.478 (width 0.3) (layer Eco1.User)
+    (gr_text "14,478 mm" (at 159.592 120.269 90) (layer Eco1.User)
       (effects (font (size 1.5 1.5) (thickness 0.3)))
     )
-    (feature1 (pts (xy 153.8 113) (xy 159.3 113)))
-    (feature2 (pts (xy 153.8 127) (xy 159.3 127)))
-    (crossbar (pts (xy 156.6 127) (xy 156.6 113)))
-    (arrow1a (pts (xy 156.6 113) (xy 157.186421 114.126504)))
-    (arrow1b (pts (xy 156.6 113) (xy 156.013579 114.126504)))
-    (arrow2a (pts (xy 156.6 127) (xy 157.186421 125.873496)))
-    (arrow2b (pts (xy 156.6 127) (xy 156.013579 125.873496)))
-  )
+    (feature1 (pts (xy 154.178 113.03) (xy 160.942 113.03)))
+    (feature2 (pts (xy 154.178 127.508) (xy 160.942 127.508)))
+    (crossbar (pts (xy 158.242 127.508) (xy 158.242 113.03)))
+    (arrow1a (pts (xy 158.242 113.03) (xy 158.828421 114.156504)))
+    (arrow1b (pts (xy 158.242 113.03) (xy 157.655579 114.156504)))
+    (arrow2a (pts (xy 158.242 127.508) (xy 158.828421 126.381496)))
+    (arrow2b (pts (xy 158.242 127.508) (xy 157.655579 126.381496)))
+  )
+  (gr_arc (start 127.762 114.3) (end 126.492 114.3) (angle 90) (layer Edge.Cuts) (width 0.15))
+  (gr_arc (start 151.638 114.3) (end 151.638 113.03) (angle 90) (layer Edge.Cuts) (width 0.15))
+  (gr_arc (start 151.638 126.238) (end 152.908 126.238) (angle 90) (layer Edge.Cuts) (width 0.15))
+  (gr_arc (start 127.762 126.238) (end 127.762 127.508) (angle 90) (layer Edge.Cuts) (width 0.15))
   (gr_line (start 143.2 116.8) (end 142.8 116.6) (layer F.SilkS) (width 0.2))
   (gr_line (start 143.2 116.8) (end 142.8 117) (layer F.SilkS) (width 0.2))
@@
   (gr_line (start 139.2 114.8) (end 139.2 113.4) (layer F.SilkS) (width 0.2))
   (gr_line (start 141.6 116.8) (end 143.2 116.8) (layer F.SilkS) (width 0.2))
-  (gr_line (start 127 114.3) (end 127 125.73) (layer Edge.Cuts) (width 0.15))
-  (gr_line (start 151.13 113.03) (end 128.27 113.03) (layer Edge.Cuts) (width 0.15))
-  (gr_line (start 152.4 125.73) (end 152.4 114.3) (layer Edge.Cuts) (width 0.15))
+  (gr_line (start 126.492 114.3) (end 126.492 126.238) (layer Edge.Cuts) (width 0.15))
+  (gr_line (start 151.638 113.03) (end 127.762 113.03) (layer Edge.Cuts) (width 0.15))
+  (gr_line (start 152.908 126.238) (end 152.908 114.3) (layer Edge.Cuts) (width 0.15))
   (gr_text "Autor: Matthias Nowak\nFür: Bertil Maier" (at 139.7 121) (layer B.SilkS)
     (effects (font (size 1.3 1.3) (thickness 0.25)))
   )
-  (gr_text "LSM6DSL Breakout" (at 139.2 117.2) (layer B.SilkS)
+  (gr_text "LSM6DSL Breakout" (at 139.446 116.586) (layer B.SilkS)
     (effects (font (size 1.5 1.5) (thickness 0.3)))
   )
@@
     (effects (font (size 1.5 1.5) (thickness 0.3)) (justify left))
   )
-  (gr_line (start 128.27 127) (end 151.13 127) (layer Edge.Cuts) (width 0.15))
+  (gr_line (start 127.762 127.508) (end 151.638 127.508) (layer Edge.Cuts) (width 0.15))
   (segment (start 139.2 117) (end 141 118.8) (width 0.2) (layer B.Cu) (net 1))
   (via (at 141 118.8) (size 0.6) (drill 0.4) (layers F.Cu B.Cu) (net 1))
